File: LoRa Environmental Sensors.kicad_pcb (KiCad board)
At the start: 2 copper layers, 5 parts, among them U1 BME280BreakoutBoard, U2 ATtiny85-20SU, U3 RFM95W-868S2

Commit message: add gerber files
Routing:
- net GND: track 7.01 -> 15.9 mm, vias 3 -> 5
Other:
- board outline added: 50 x 25 mm
Changed lines of the file:
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@@
-(kicad_pcb (version 20171130) (host pcbnew 5.0.0+dfsg1-2)
+(kicad_pcb (version 20171130) (host pcbnew "(5.0.1)-4")
   (general
     (thickness 1.6)
     (drawings 5)
-    (tracks 46)
+    (tracks 49)
     (zones 0)
     (modules 5)
@@
   (layers
     (0 F.Cu signal)
-    (31 B.Cu signal)
+    (31 B.Cu signal hide)
     (32 B.Adhes user)
     (33 F.Adhes user)
@@
     (trace_min 0.1524)
     (segment_width 0.2)
-    (edge_width 0.15)
+    (edge_width 0.2)
     (via_size 0.762)
     (via_drill 0.381)
@@
     (pad_drill 0.762)
     (pad_to_mask_clearance 0.0508)
+    (solder_mask_min_width 0.25)
     (aux_axis_origin 0 0)
-    (visible_elements FFFFFF7F)
+    (visible_elements 7FFFFFFF)
     (pcbplotparams
-      (layerselection 0x010fc_ffffffff)
-      (usegerberextensions false)
+      (layerselection 0x010f0_ffffffff)
+      (usegerberextensions true)
       (usegerberattributes false)
       (usegerberadvancedattributes false)
@@
       (psa4output false)
       (plotreference true)
-      (plotvalue true)
+      (plotvalue false)
       (plotinvisibletext false)
       (padsonsilk false)
@@
       (outputformat 1)
       (mirror false)
-      (drillshape 1)
+      (drillshape 0)
       (scaleselection 1)
-      (outputdirectory ""))
+      (outputdirectory "gerbers/"))
   )
   (net 0 "")
@@
   )
   (gr_text "LoRa Environmental Sensors\nRev. 01" (at 176.784 70.993 90) (layer B.SilkS)
-    (effects (font (size 0.508 0.508) (thickness 0.03175)) (justify mirror))
-  )
-  (gr_line (start 178.143 64.984) (end 128.143 64.984) (layer F.SilkS) (width 0.2))
-  (gr_line (start 178.143 64.984) (end 178.143 89.984) (layer F.SilkS) (width 0.2))
-  (gr_line (start 128.143 89.984) (end 178.143 89.984) (layer F.SilkS) (width 0.2))
-  (gr_line (start 128.143 64.984) (end 128.143 89.984) (layer F.SilkS) (width 0.2))
+    (effects (font (size 0.508 0.508) (thickness 0.03175)))
+  )
+  (gr_line (start 178.143 64.984) (end 128.143 64.984) (layer Edge.Cuts) (width 0.2))
+  (gr_line (start 178.143 64.984) (end 178.143 89.984) (layer Edge.Cuts) (width 0.2))
+  (gr_line (start 128.143 89.984) (end 178.143 89.984) (layer Edge.Cuts) (width 0.2))
+  (gr_line (start 128.143 64.984) (end 128.143 89.984) (layer Edge.Cuts) (width 0.2))
   (via (at 134.112 83.439) (size 0.762) (drill 0.381) (layers F.Cu B.Cu) (net 1))
   (segment (start 134.097 85.724) (end 134.097 83.454) (width 0.762) (layer F.Cu) (net 1))
@@
   (segment (start 146.097 69.724) (end 146.097 71.835) (width 0.762) (layer F.Cu) (net 1))
   (segment (start 146.097 71.835) (end 146.05 71.882) (width 0.762) (layer F.Cu) (net 1))
+  (via (at 151.13 69.85) (size 0.762) (drill 0.381) (layers F.Cu B.Cu) (net 1))
+  (via (at 160.02 69.85) (size 0.762) (drill 0.381) (layers F.Cu B.Cu) (net 1))
+  (segment (start 151.13 69.85) (end 160.02 69.85) (width 0.762) (layer F.Cu) (net 1))
   (segment (start 143.129 66.485) (end 140.335 66.485) (width 0.254) (layer B.Cu) (net 2))
   (segment (start 158.56 88.455) (end 164.211 82.804) (width 0.762) (layer B.Cu) (net 2))
@@
     (polygon
       (pts
-        (xy 127.889 90.424) (xy 178.435 90.297) (xy 178.435 64.77) (xy 127.889 64.77)
+        (xy 127 90.17) (xy 179.07 90.17) (xy 179.07 63.5) (xy 127 63.5)
       )
     )

Commit message: update pcb
Parts:
- moved U2 10.9 mm to (160.1, 81.8), turned to 180 degrees
- moved U3 1.78 mm to (139.3, 77.6), turned to 270 degrees
- turned U1 to 0 degrees
Routing:
- net /NSS: track 17.6 -> 28.1 mm
- net /SCK: track 30.8 -> 41.3 mm
- net VCC: track 65.5 -> 58.0 mm
- net /MOSI: track 32.8 -> 37.7 mm
- net /CS: track 13.3 -> 16.3 mm
- net GND: track 15.9 -> 17.9 mm, vias 5 -> 7
- net /MISO: track 34.1 -> 34.7 mm

Commit message: update gerbers
Other:
- board text added: "ANA"
Changed lines of the file:
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@@
-(kicad_pcb (version 20171130) (host pcbnew 5.0.0+dfsg1-2)
+(kicad_pcb (version 20171130) (host pcbnew "(5.0.1)-4")
   (general
     (thickness 1.6)
-    (drawings 5)
+    (drawings 6)
     (tracks 64)
     (zones 0)
@@
   (layers
     (0 F.Cu signal)
-    (31 B.Cu signal)
-    (32 B.Adhes user)
-    (33 F.Adhes user)
-    (34 B.Paste user)
-    (35 F.Paste user)
-    (36 B.SilkS user)
+    (31 B.Cu signal hide)
+    (32 B.Adhes user hide)
+    (33 F.Adhes user hide)
+    (34 B.Paste user hide)
+    (35 F.Paste user hide)
+    (36 B.SilkS user hide)
     (37 F.SilkS user)
-    (38 B.Mask user)
+    (38 B.Mask user hide)
     (39 F.Mask user)
-    (40 Dwgs.User user)
-    (41 Cmts.User user)
-    (42 Eco1.User user)
-    (43 Eco2.User user)
-    (44 Edge.Cuts user)
-    (45 Margin user)
-    (46 B.CrtYd user)
-    (47 F.CrtYd user)
-    (48 B.Fab user)
-    (49 F.Fab user)
+    (40 Dwgs.User user hide)
+    (41 Cmts.User user hide)
+    (42 Eco1.User user hide)
+    (43 Eco2.User user hide)
+    (44 Edge.Cuts user hide)
+    (45 Margin user hide)
+    (46 B.CrtYd user hide)
+    (47 F.CrtYd user hide)
+    (48 B.Fab user hide)
+    (49 F.Fab user hide)
   )
   (setup
-    (last_trace_width 0.762)
+    (last_trace_width 0.254)
     (user_trace_width 0.762)
     (trace_clearance 0.254)
@@
       (xy 0.036301 3.553379) (xy 0.050473 3.546591)) (layer B.SilkS) (width 0.01))
   )
+  (gr_text ANA (at 132.08 82.55 90) (layer F.SilkS)
+    (effects (font (size 1 1) (thickness 0.25)))
+  )
   (gr_text "LoRa Environmental Sensors\nRev. 01" (at 176.784 70.993 90) (layer B.SilkS)

Commit message: update gerber files
Parts:
- moved G*** 18.5 mm to (171.6, 86.6)
Changed lines of the file:
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@@
-(kicad_pcb (version 20171130) (host pcbnew "(5.0.1)-4")
+(kicad_pcb (version 20171130) (host pcbnew 5.0.0+dfsg1-2)
   (general
     (thickness 1.6)
@@
   (layers
     (0 F.Cu signal)
-    (31 B.Cu signal hide)
-    (32 B.Adhes user hide)
-    (33 F.Adhes user hide)
-    (34 B.Paste user hide)
-    (35 F.Paste user hide)
-    (36 B.SilkS user hide)
+    (31 B.Cu signal)
+    (32 B.Adhes user)
+    (33 F.Adhes user)
+    (34 B.Paste user)
+    (35 F.Paste user)
+    (36 B.SilkS user)
     (37 F.SilkS user)
-    (38 B.Mask user hide)
+    (38 B.Mask user)
     (39 F.Mask user)
-    (40 Dwgs.User user hide)
-    (41 Cmts.User user hide)
-    (42 Eco1.User user hide)
-    (43 Eco2.User user hide)
-    (44 Edge.Cuts user hide)
-    (45 Margin user hide)
-    (46 B.CrtYd user hide)
-    (47 F.CrtYd user hide)
-    (48 B.Fab user hide)
-    (49 F.Fab user hide)
+    (40 Dwgs.User user)
+    (41 Cmts.User user)
+    (42 Eco1.User user)
+    (43 Eco2.User user)
+    (44 Edge.Cuts user)
+    (45 Margin user)
+    (46 B.CrtYd user)
+    (47 F.CrtYd user)
+    (48 B.Fab user)
+    (49 F.Fab user)
   )
   (setup
@@
       (layerselection 0x010f0_ffffffff)
       (usegerberextensions true)
-      (usegerberattributes false)
+      (usegerberattributes true)
       (usegerberadvancedattributes false)
       (creategerberjobfile false)
       (excludeedgelayer true)
-      (linewidth 0.100000)
+      (linewidth 0.150000)
       (plotframeref false)
       (viasonmask false)
@@
   )
   (module graphic:spielhuus (layer B.Cu)
-    (at 171.069 68.072 270)
+    (at 171.577 86.614 270)
     (fp_text reference G*** (at 0 0 270) (layer B.SilkS) hide
       (effects (font (size 1.524 1.524) (thickness 0.3)) (justify mirror))
@@
     (effects (font (size 1 1) (thickness 0.25)))
   )
-  (gr_text "LoRa Environmental Sensors\nRev. 01" (at 176.784 70.993 90) (layer B.SilkS)
+  (gr_text "LoRa Environmental Sensors\nRev. 01" (at 176.53 83.566 90) (layer B.SilkS)
     (effects (font (size 0.508 0.508) (thickness 0.03175)))
   )
